Commit message: added br2 files from blue

File: description/robot.urdf.xacro (robot description, xacro)
@@ -2,3 +2,6 @@
 <robot xmlns:xacro="http://www.ros.org/wiki/xacro"  name="robot">
     <xacro:include filename="robot_core.xacro" />
+    <!-- <xacro:include filename="gazebo_control.xacro" /> -->
+    <!-- <xacro:include filename="ros2_control.xacro" /> -->
+    <xacro:include filename="camera.xacro" />
 </robot>

File: description/robot_core.xacro (robot description, xacro)
@@ -55,4 +55,7 @@
         </xacro:inertial_box>
   </link>
+  <gazebo reference="chassis">
+    <material>Gazebo/White</material>
+  </gazebo>
   <!-- LEFT WHEEL LINK -->
   <joint name="left_wheel_joint" type="continuous">
@@ -78,4 +81,7 @@
     </xacro:inertial_cylinder>
   </link>
+   <gazebo reference="left_wheel">
+    <material>Gazebo/Blue</material>
+  </gazebo>
   <!-- RIGHT WHEEL -->
   <joint name="right_wheel_joint" type="continuous">
@@ -97,5 +103,11 @@
       </geometry>
     </collision>
+    <xacro:inertial_cylinder mass="${wheel_mass}" length="${wheel_thickness}" radius="${wheel_radius}">
+            <origin xyz="0 0 0" rpy="0 0 0"/>
+    </xacro:inertial_cylinder>
   </link>
+   <gazebo reference="right_wheel">
+    <material>Gazebo/Blue</material>
+  </gazebo>
   <!-- CASTER WHEEL LINK -->
   <joint name="caster_wheel_joint" type="fixed">
@@ -120,3 +132,6 @@
         </xacro:inertial_sphere>
   </link>
+  <gazebo reference="caster_wheel">
+    <material>Gazebo/Black</material>
+  </gazebo>
 </robot>
